Commit message: Add configuration files and teleop bridge for dual arm control
- Created `ompl_planning.yaml` for OMPL planner configurations for xArm and UF arms.
- Added `ros2_controllers.yaml` to define controllers for xArm, UF, RG6 gripper, and slider.
- Introduced `sensors_3d.yaml.disabled` for 3D sensor configuration using occupancy map monitor.
- Added `uf_servo.yaml` and `xarm_servo.yaml` for servo configurations of UF850 and xArm5 respectively.
- Implemented `teleop_bridge.py` for joystick control, including smooth velocity handling and arm switching.

File: dual_arm_moveit_config/config/dual_arm_world.urdf.xacro (robot description, xacro)
@@ -4,5 +4,5 @@
 <!-- |    EDITING THIS FILE BY HAND IS NOT RECOMMENDED                                 | -->
 <!-- =================================================================================== -->
-<robot name="dual_arm_disassembly_cell">
+<robot name="dual_arm_disassembly_cell" xmlns:xacro="http://www.ros.org/wiki/xacro">
   <!-- ================================================= -->
   <!-- Arguments                                         -->
@@ -930,80 +930,115 @@
     <origin rpy="0 0 0" xyz="0.461 -0.292 0.837"/>
   </joint>
+  <xacro:arg name="hw_type" default="fake"/>
   <ros2_control name="DualArmControl" type="system">
     <hardware>
-      <plugin>mock_components/GenericSystem</plugin>
-      <plugin>topic_based_ros2_control/TopicBasedSystem</plugin>
-      <param name="joint_commands_topic">/robot_joint_commands</param>
-      <param name="joint_states_topic">/robot_joint_states</param>
-      <param name="trigger_joint_command_threshold">-1</param> </hardware>
-      <!-- <plugin>isaac_ros2_control/IsaacSystem</plugin>
-      <param name="joint_commands_topic">/isaac_joint_commands</param>
-      <param name="joint_states_topic">/isaac_joint_states</param> -->
+      <xacro:if value="${'$(arg hw_type)' == 'fake'}">
+        <plugin>mock_components/GenericSystem</plugin>
+      </xacro:if>
+      <xacro:if value="${'$(arg hw_type)' == 'real'}">
+        <plugin>topic_based_ros2_control/TopicBasedSystem</plugin>
+        <param name="joint_commands_topic">/robot_joint_commands</param>
+        <param name="joint_states_topic">/robot_joint_states</param>
+        <param name="trigger_joint_command_threshold">-1</param>
+      </xacro:if>
+      <xacro:if value="${'$(arg hw_type)' == 'isaac'}">
+        <plugin>isaac_ros2_control/IsaacSystem</plugin>
+        <param name="joint_commands_topic">/isaac_joint_commands</param>
+        <param name="joint_states_topic">/isaac_joint_states</param>
+      </xacro:if>
     </hardware>
     <joint name="slider_slider_joint">
       <command_interface name="position"/>
-      <state_interface name="position"><param name="initial_value">0.0</param></state_interface>
+      <state_interface name="position">
+        <xacro:if value="${'$(arg hw_type)' == 'fake'}">
+          <param name="initial_value">0.0</param>
+        </xacro:if>
+      </state_interface>
       <state_interface name="velocity"/>
     </joint>
     <joint name="xarm5_joint1">
       <command_interface name="position"/>
-      <state_interface name="position"><param name="initial_value">0.0</param></state_interface>
+      <state_interface name="position">
+        <xacro:if value="${'$(arg hw_type)' == 'fake'}"><param name="initial_value">0.0</param></xacro:if>
+      </state_interface>
       <state_interface name="velocity"/>
     </joint>
     <joint name="xarm5_joint2">
       <command_interface name="position"/>
-      <state_interface name="position"><param name="initial_value">0.0</param></state_interface>
+      <state_interface name="position">
+        <xacro:if value="${'$(arg hw_type)' == 'fake'}"><param name="initial_value">0.0</param></xacro:if>
+      </state_interface>
       <state_interface name="velocity"/>
     </joint>
     <joint name="xarm5_joint3">
       <command_interface name="position"/>
-      <state_interface name="position"><param name="initial_value">-1.5708</param></state_interface>
+      <state_interface name="position">
+        <xacro:if value="${'$(arg hw_type)' == 'fake'}"><param name="initial_value">-1.5708</param></xacro:if>
+      </state_interface>
       <state_interface name="velocity"/>
     </joint>
     <joint name="xarm5_joint4">
       <command_interface name="position"/>
-      <state_interface name="position"><param name="initial_value">1.5708</param></state_interface>
+      <state_interface name="position">
+        <xacro:if value="${'$(arg hw_type)' == 'fake'}"><param name="initial_value">1.5708</param></xacro:if>
+      </state_interface>
       <state_interface name="velocity"/>
     </joint>
     <joint name="xarm5_joint5">
       <command_interface name="position"/>
-      <state_interface name="position"><param name="initial_value">0.0</param></state_interface>
+      <state_interface name="position">
+        <xacro:if value="${'$(arg hw_type)' == 'fake'}"><param name="initial_value">0.0</param></xacro:if>
+      </state_interface>
       <state_interface name="velocity"/>
     </joint>
     <joint name="u1_joint1">
       <command_interface name="position"/>
-      <state_interface name="position"><param name="initial_value">0.0</param></state_interface>
+      <state_interface name="position">
+        <xacro:if value="${'$(arg hw_type)' == 'fake'}"><param name="initial_value">0.0</param></xacro:if>
+      </state_interface>
       <state_interface name="velocity"/>
     </joint>
     <joint name="u1_joint2">
       <command_interface name="position"/>
-      <state_interface name="position"><param name="initial_value">0.0</param></state_interface>
+      <state_interface name="position">
+        <xacro:if value="${'$(arg hw_type)' == 'fake'}"><param name="initial_value">0.0</param></xacro:if>
+      </state_interface>
       <state_interface name="velocity"/>
     </joint>
     <joint name="u1_joint3">
       <command_interface name="position"/>
-      <state_interface name="position"><param name="initial_value">-1.5708</param></state_interface>
+      <state_interface name="position">
+        <xacro:if value="${'$(arg hw_type)' == 'fake'}"><param name="initial_value">-1.5708</param></xacro:if>
+      </state_interface>
       <state_interface name="velocity"/>
     </joint>
     <joint name="u1_joint4">
       <command_interface name="position"/>
-      <state_interface name="position"><param name="initial_value">0.0</param></state_interface>
+      <state_interface name="position">
+        <xacro:if value="${'$(arg hw_type)' == 'fake'}"><param name="initial_value">0.0</param></xacro:if>
+      </state_interface>
       <state_interface name="velocity"/>
     </joint>
     <joint name="u1_joint5">
       <command_interface name="position"/>
-      <state_interface name="position"><param name="initial_value">-1.5708</param></state_interface>
+      <state_interface name="position">
+        <xacro:if value="${'$(arg hw_type)' == 'fake'}"><param name="initial_value">-1.5708</param></xacro:if>
+      </state_interface>
       <state_interface name="velocity"/>
     </joint>
     <joint name="u1_joint6">
       <command_interface name="position"/>
-      <state_interface name="position"><param name="initial_value">0.0</param></state_interface>
+      <state_interface name="position">
+        <xacro:if value="${'$(arg hw_type)' == 'fake'}"><param name="initial_value">0.0</param></xacro:if>
+      </state_interface>
       <state_interface name="velocity"/>
     </joint>
     <joint name="rg6_l_out">
       <command_interface name="position"/>
-      <state_interface name="position"><param name="initial_value">0.0</param></state_interface>
-      <state_interface name="velocity"/>
-    </joint>
-    </ros2_control>
+      <state_interface name="position">
+        <xacro:if value="${'$(arg hw_type)' == 'fake'}"><param name="initial_value">0.0</param></xacro:if>
+      </state_interface>
+      <state_interface name="velocity"/>
+    </joint>
+  </ros2_control>
 </robot>
