Commit message: feat: Add vision training notebooks and project configs, excluding large binary artifacts

File: dual_arm_moveit_config/config/dual_arm_world.urdf (robot description, URDF)
Before this commit: robot dual_arm_disassembly_cell, 36 links, 35 joints
Links:
- link ft_ft300_mounting_plate: geometry collision mesh filename=file:///home/adip/workspace/disassembly_ws/install/robotiq_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; visual mesh filename=file:///home/adip/workspace/disassembly_ws/install/robotiq_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
- link ft_ft300_sensor: geometry collision mesh filename=file:///home/adip/workspace/disassembly_ws/install/robotiq_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; visual mesh filename=file:///home/adip/workspace/disassembly_ws/install/robotiq_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

File: dual_arm_moveit_config/config/dual_arm_world.urdf.xacro (robot description, xacro)
@@ -1,5 +1,5 @@
 <?xml version="1.0" ?>
 <!-- =================================================================================== -->
-<!-- |    This document was autogenerated by xacro from /home/adip/workspaces/disassembly_ws/src/scene_description/urdf/dual_arm_scene.urdf.xacro | -->
+<!-- |    This document was autogenerated by xacro from /home/adip/workspace/disassembly_ws/src/scene_description/urdf/dual_arm_scene.urdf.xacro | -->
 <!-- |    EDITING THIS FILE BY HAND IS NOT RECOMMENDED                                 | -->
 <!-- =================================================================================== -->
@@ -315,5 +315,5 @@
       <origin rpy="0 0 0" xyz="0 0 0"/>
       <geometry>
-        <mesh filename="file:///home/adip/workspaces/disassembly_ws/install/robotiq_ft_sensor_description/share/robotiq_ft_sensor_description/meshes/visual/robotiq_ft300.STL"/>
+        <mesh filename="file:///home/adip/workspace/disassembly_ws/install/robotiq_ft_sensor_description/share/robotiq_ft_sensor_description/meshes/visual/robotiq_ft300.STL"/>
       </geometry>
       <material name="Robotiq-Black">
@@ -324,5 +324,5 @@
       <origin rpy="0 0 0" xyz="0 0 0"/>
       <geometry>
-        <mesh filename="file:///home/adip/workspaces/disassembly_ws/install/robotiq_ft_sensor_description/share/robotiq_ft_sensor_description/meshes/collision/robotiq_ft300.STL"/>
+        <mesh filename="file:///home/adip/workspace/disassembly_ws/install/robotiq_ft_sensor_description/share/robotiq_ft_sensor_description/meshes/collision/robotiq_ft300.STL"/>
       </geometry>
     </collision>
@@ -333,5 +333,5 @@
       <origin rpy="0 0 0" xyz="0 0 0"/>
       <geometry>
-        <mesh filename="file:///home/adip/workspaces/disassembly_ws/install/robotiq_ft_sensor_description/share/robotiq_ft_sensor_description/meshes/visual/mountings/robotiq_ft300-G-062-COUPLING_G-50-4M6-1D6_20181119.STL"/>
+        <mesh filename="file:///home/adip/workspace/disassembly_ws/install/robotiq_ft_sensor_description/share/robotiq_ft_sensor_description/meshes/visual/mountings/robotiq_ft300-G-062-COUPLING_G-50-4M6-1D6_20181119.STL"/>
       </geometry>
       <material name="Robotiq-Grey">
@@ -342,5 +342,5 @@
       <origin rpy="0 0 0" xyz="0 0 0"/>
       <geometry>
-        <mesh filename="file:///home/adip/workspaces/disassembly_ws/install/robotiq_ft_sensor_description/share/robotiq_ft_sensor_description/meshes/collision/mountings/robotiq_ft300-G-062-COUPLING_G-50-4M6-1D6_20181119.STL"/>
+        <mesh filename="file:///home/adip/workspace/disassembly_ws/install/robotiq_ft_sensor_description/share/robotiq_ft_sensor_description/meshes/collision/mountings/robotiq_ft300-G-062-COUPLING_G-50-4M6-1D6_20181119.STL"/>
       </geometry>
     </collision>

File: scene_description/urdf/scene.urdf (robot description, URDF)
Before this commit: robot scene, 2 links, 1 joints
Links:
- link base_link: geometry collision mesh filename=file:///home/adip/workspace/disassembly_ws/src/scene_descri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 scale=0.001 0.001 0.001; visual mesh filename=file:///home/adip/workspace/disassembly_ws/src/scene_descri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 scale=0.001 0.001 0.001
